File: CopyBoard64/CopyBoard64.brd (EAGLE design)
At the start: 49.5 x 49.5 mm, 10 parts, among them CN1 COMMODORE, CN2 READ, CN3 WRITE, IC1 74LS14

Commit message: Updated CopyBoard64 project files
Parts:
- moved C1 19.0 mm to (15.2, 20.3), turned to 90 degrees
- moved IC1 3.81 mm to (26.7, 20.3), turned to 0 degrees
- moved LOGO1 0.90 mm to (23.1, 32.4)
Routing:
- net VCC: track 99.0 -> 114.4 mm, vias 4 -> 5
- net INVREAD: track 44.8 -> 56.9 mm
- net LEDA2: track 25.4 -> 17.3 mm
- net READ: track 61.4 -> 53.5 mm, vias 3 -> 2
- net GND: track 119.0 -> 114.5 mm, vias 3 -> 4
- net MOTOR: track 87.8 -> 85.2 mm
- net SENSE: track 42.4 -> 41.9 mm
