File: 27CXXX/27CXXX-Double.brd (EAGLE design)
At the start: 100.3 x 92.7 mm, 14 parts, among them IC1 27C4096, IC2 27C400/800/160, IC3 27C4096, IC4 27C400/800/160, SW1 A18, SW2 A19, SW3 A18, SW4 A19

Commit message: Updated 27CXXX Design Files
Parts:
- IC2, IC4: device sj_ic:ZIF42 -> sj_ic:ZIF42F
- moved R1 7.62 mm to (31.1, 92.1)
- moved R2 7.62 mm to (46.4, 92.1)
- moved R3 7.62 mm to (81.9, 92.1)
- moved R4 7.62 mm to (97.2, 92.1)
- moved SW1 7.62 mm to (35.6, 92.1)
- moved SW2 7.62 mm to (41.9, 92.1)
- moved SW3 7.62 mm to (86.4, 92.1)
- moved SW4 7.62 mm to (92.7, 92.1)
Routing:
- net VCC: track 126.9 -> 141.4 mm
- net VCC1: track 126.9 -> 141.4 mm
- net A39: track 19.0 -> 30.4 mm
- net A18: track 19.0 -> 30.4 mm
- net A19: track 19.0 -> 30.4 mm
- net A38: track 19.0 -> 30.4 mm
- net GND1: track 218.7 -> 226.3 mm
- net GND: track 218.7 -> 226.3 mm
Other:
- board size 100.3 x 92.7 mm -> 100.3 x 100.3 mm
