File: 27CXXX/27CXXX.brd (EAGLE design)
At the start: 49.5 x 82.5 mm, 7 parts, among them IC1 27C4096, IC2 27C400/800/160, SW1 A18, SW2 A19

Commit message: Updated 27CXXX Design Files
Parts:
- IC2: device sj_ic:DIP42W -> sj_ic:ZIF42F
- moved SW1 17.2 mm to (35.6, 92.1)
- moved SW2 17.2 mm to (41.9, 92.1)
- moved R1 17.1 mm to (31.1, 92.1)
- moved R2 17.1 mm to (46.4, 92.1)
- moved LOGO1 6.48 mm to (11.0, 5.08)
Routing:
- net VCC: track 107.9 -> 141.4 mm
- net A19: track 8.89 -> 30.4 mm
- net A18: track 10.2 -> 30.4 mm
- net GND: track 209.2 -> 226.3 mm
- net Q15: track 121.0 -> 120.2 mm
- net Q11: track 52.4 -> 52.9 mm
Other:
- board size 49.5 x 82.5 mm -> 49.5 x 100.3 mm
