File: 27CXXX/27CXXX.sch (EAGLE design)
At the start: 6 parts, among them IC1 27C4096, IC2 27C400/800/160, SW1 A18, SW2 A19

Commit message: Updated 27CXXX Design Files
Parts:
- IC2: device sj_ic:27C160_DIP -> sj_ic:27C160_ZIF42F
Changed lines of the file:
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@@
 </part>
 <part name="IC1" library="sj_ic" deviceset="27C4096" device="_DIP" value="27C4096"/>
-<part name="IC2" library="sj_ic" deviceset="27C160" device="_DIP" value="27C400/800/160"/>
+<part name="IC2" library="sj_ic" deviceset="27C160" device="_ZIF42F" value="27C400/800/160"/>
 <part name="VCC1" library="sj_standart" deviceset="SUPPLY_VCC" device="" value="VCC"/>
 <part name="GND1" library="sj_standart" deviceset="SUPPLY_GND" device="" value="GND"/>
